File: furnace_power/furnace_power.kicad_sch (KiCad schematic)
At the start: 0 parts

Commit message: Started main schematic.
Parts:
- added C1: 300uF, Capacitor_THT:CP_Radial_D13.0mm_P7.50mm, symbol Device:C
- added C2: C, Capacitor_SMD:C_0603_1608Metric_Pad1.08x0.95mm_HandSolder, symbol Device:C
- added D1: model_+_max_current, Diode_THT:Diode_Bridge_Vishay_KBU, symbol Diode_Bridge:KBU4G
- added J1: Conn_01x03_Pin, Connector_Phoenix_MC:PhoenixContact_MCV_1,5_3-G-3.81_1x03_P3.81mm_Vertical, symbol Connector:Conn_01x03_Pin
- added Q1: C3M0120090D, Package_TO_SOT_THT:TO-247-3_Vertical, symbol Transistor_FET:C3M0120090D
- added R1: R_gate_not_fited, Resistor_SMD:R_0603_1608Metric_Pad0.98x0.95mm_HandSolder, symbol Device:R
- added R2: 0.1_1210_sense, Resistor_SMD:R_1210_3225Metric, symbol Device:R
- added RV1: 420V, Varistor:RV_Disc_D7mm_W5.7mm_P5mm, symbol Device:Varistor
- added TP1, TP2: HeatSink, Connector_Pin:Pin_D1.3mm_L11.0mm_LooseFit, symbol Connector:TestPoint
- added TP3: PWM, Connector_Pin:Pin_D1.3mm_L11.0mm_LooseFit, symbol Connector:TestPoint
- added TP4: 20VDC, Connector_Pin:Pin_D1.3mm_L11.0mm_LooseFit, symbol Connector:TestPoint
- added TP5: TP, Connector_Pin:Pin_D1.3mm_L11.0mm_LooseFit, symbol Connector:TestPoint
- added U1: FAN3111E, Package_TO_SOT_SMD:SOT-23-5, symbol Driver_FET:FAN3111E
Connections:
- new net: C1.2, D1.4 (-)
- new net: R1.1, U1.5 (OUT)
- new net: Q1.1 (G), R1.2, TP5.1
- new net: Q1.3 (S), R2.1
- new net +20DC: C2.1, TP4.1, U1.1 (VDD)
- new net +320DC: C1.1, D1.1 (+), Q1.2 (D)
- new net GND: C2.2, R2.2, U1.2 (GND)
- new net L: D1.3, J1.1 (Pin_1), RV1.1
- new net N: D1.2, J1.2 (Pin_2), RV1.2
- new net PE: J1.3 (Pin_3), TP1.1, TP2.1
- new net PWM: TP3.1, U1.3 (IN+)
- no-connect marks 0 -> 1
Other:
- note added: "230AC to 320DC section"
