File: main_power/pico_gate_driver.kicad_sch (KiCad schematic)
At the start: 1 part

Commit message: repo cleaning
Parts:
- removed U?: Pico, RPi_Pico:RPi_Pico_SMD_TH, symbol MCU_RaspberryPi_and_Boards:Pico
- added C? (x4): C, symbol Device:C
- added C? (x2): 100n, symbol Device:C
- added C? (x2): 1u, symbol Device:C
- added D? (x2): D_Filled, symbol Device:D_Filled
- added D?: D_Small_Filled, symbol Device:D_Small_Filled
- added IC? (x2): UCC27512DRSR, SON95P300X300X80-7N-D, symbol UCC27512DRSR:UCC27512DRSR
- added Q? (x4): REPLACE, Package_SO:Vishay_PowerPAK_1212-8_Single, symbol Transistor_FET:SiS454DN
- added R? (x4): R, symbol Device:R
- added R? (x2): option_DNM, symbol Device:R_Small
- added R? (x2): 0, symbol Device:R_Small
- added R? (x6): R_Small, symbol Device:R_Small
- added TP?: SW_GATE, symbol Connector:TestPoint
- added TP?: LO_Gate, symbol Connector:TestPoint
- added TP?: HO_Gate, symbol Connector:TestPoint
- added TP? (x2): TestPoint, symbol Connector:TestPoint
- added U?: NSL-32, OptoDevice:Luna_NSL-32, symbol Isolator:NSL-32
- added U?: UCC27714DR, Package_SO:SOIC-14_3.9x8.7mm_P1.27mm, symbol Driver_FET:UCC27714D
Connections:
- new net: D?.2 (A), Q?.4 (G), R?.1, R?.2, TP?.1
- new net: C?.1, R?.1, R?.2, U?.7 (VDD)
- new net: Q?.4 (G), R?.1, R?.2, TP?.1 (x2)
- new net: D?.1 (K), R?.1, U?.6 (LO)
- new net: D?.2 (A), Q?.4 (G), R?.2, R?.2, TP?.1
- new net: IC?.6 (IN-), R?.2 (x2)
- new net: IC?.4 (OUT), R?.1 (x2)
- new net: C?.1, D?.1 (K), U?.13 (HB)
- new net: D?.2 (A), R?.2
- new net: D?.1 (K), R?.1, U?.12 (HO)
- new net +18DC: C?.1, C?.1, C?.1, C?.2, IC?.3 (VDD), IC?.3 (VDD), Q?.5 (D), R?.1
- new net GND: C?.1, C?.2, C?.2, C?.2, C?.2, C?.2, C?.2, IC?.2 (GND_1), IC?.2 (GND_1), IC?.5 (GND_2), IC?.5 (GND_2), IC?.7 (EP), IC?.7 (EP), Q?.1 (S), Q?.1 (S), Q?.1 (S), Q?.2 (S), Q?.2 (S), Q?.2 (S), Q?.3 (S), Q?.3 (S), Q?.3 (S), R?.1, R?.1, R?.1, R?.2, R?.2, U?.2 (K), U?.3 (VSS), U?.5 (COM)
- new net MCU_ENABLE: U?.4 (EN/NC)
- new net MCU_NPWM_A: R?.1
- new net MCU_PWM_A: R?.1
- new net NPWM: C?.1, R?.2, U?.2 (LI)
- new net PWM: C?.1, R?.2, U?.1 (HI)
- new net PWM_B: IC?.1 (IN+)
- new net PWM_C: IC?.1 (IN+)
- new net SW: C?.2, Q?.1 (S), Q?.2 (S), Q?.3 (S), Q?.5 (D), R?.2, TP?.1, U?.1 (A), U?.11 (HS)
- no-connect marks 3 -> 0
Other:
- note added: "Jezeli chce zostawic opcje na inverting -> trzeba dać też zworki na in+ można też użyć zwykłcyh jumper na goldpin"
- note added: "Jezeli dowiem sie ze te r i c potrzebne -> dodać do mniejszego drivera"
- note added: "rezysotry 0h na sekcje?"

Commit message: schematic of flyback v1
Parts:
- gave numbers to parts that had none: 38
